Commit message: new

File: robot_urdf/urdf/robot4.xacro (robot description, xacro)
@@ -115,15 +115,37 @@
     <joint_properties damping="1.0" friction="1.0"/>
   </joint>
-  <link name="camera_link">
+ <link name="camera_link_connection">
 	    <collision>
-	      <origin xyz="0 0 0.025" rpy="0 0 0"/>
+	      <origin xyz="0 0 0.1" rpy="0 0 0"/>
 	      <geometry>
-		<box size="0.05 0.05 0.05"/>
+		<box size="0.1 0.1 0.25"/>
 	      </geometry>
 	    </collision>
 	    <visual>
-	      <origin xyz="0 0 0.025" rpy="0 0 0"/>
+	      <origin xyz="0 0 0.1" rpy="0 0 0"/>
 	      <geometry>
-		<box size="0.05 0.05 0.05"/>
+		<box size="0.05 0.05 0.25"/>
+	      </geometry>
+	      <material name="red">
+		<color rgba="1 0 0 1"/>
+	      </material>
+	    </visual>
+	    <inertial>
+	      <mass value="1e-5" />
+	      <origin xyz="0 0 0" rpy="0 0 0"/>
+	      <inertia ixx="1e-6" ixy="0" ixz="0" iyy="1e-6" iyz="0" izz="1e-6" />
+	    </inertial>
+  </link>
+  <link name="camera_link">
+	    <collision>
+	      <origin xyz="0 0 0" rpy="0 0 0"/>
+	      <geometry>
+		<box size="0.07 0.07 0.07"/>
+	      </geometry>
+	    </collision>
+	    <visual>
+	      <origin xyz="0 0 0" rpy="0 0 0"/>
+	      <geometry>
+		<box size="0.07 0.07 0.07"/>
 	      </geometry>
 	      <material name="red">
@@ -139,7 +161,13 @@
   <joint name="camera_joint" type="fixed">
 	    <axis xyz="0 0 1" />
-	    <origin xyz="0.23 0 0" rpy="0 0 0"/>
-	    <parent link="link_chassis"/>
+	    <origin xyz="0 0 0.27" rpy="0 0 0"/>
+	    <parent link="camera_link_connection"/>
 	    <child link="camera_link"/>
 	 </joint>
+  <joint name="camera_link_joint" type="fixed">
+	    <axis xyz="0 0 1" />
+	    <origin xyz="0.2 0 0.05" rpy="0 0 0"/>
+	    <parent link="link_chassis"/>
+	    <child link="camera_link_connection"/>
+	 </joint>
 </robot>

Commit message: funziona

File: robot_urdf/urdf/robot4.xacro (robot description, xacro)
@@ -171,3 +171,13 @@
 	    <child link="camera_link_connection"/>
 	 </joint>
+   <transmission name="cam_trans">
+      <type>transmission_interface/SimpleTransmission</type>
+      <joint name="camera_joint">
+      <hardwareInterface>hardwareInterface/EffortJointInterface</hardwareInterface>
+      </joint>
+      <actuator name="motor_cam">
+        <hardwareInterface>hardwareInterface/EffortJointInterface</hardwareInterface>
+        <mechanicalReduction>1</mechanicalReduction>
+      </actuator>
+   </transmission>
 </robot>

Commit message: new_version

File: robot_urdf/urdf/robot4.xacro (robot description, xacro)
@@ -159,5 +159,5 @@
 	    </inertial>
   </link>
-  <joint name="camera_joint" type="fixed">
+  <joint name="camera_joint" type="continuous">
 	    <axis xyz="0 0 1" />
 	    <origin xyz="0 0 0.27" rpy="0 0 0"/>

Commit message: Finito pub non funziona

File: robot_urdf/urdf/robot4.xacro (robot description, xacro)
@@ -117,13 +117,13 @@
  <link name="camera_link_connection">
 	    <collision>
-	      <origin xyz="0 0 0.1" rpy="0 0 0"/>
+	      <origin xyz="0 0 0.05" rpy="0 0 0"/>
 	      <geometry>
-		<box size="0.1 0.1 0.25"/>
+		<box size="0.05 0.05 0.15"/>
 	      </geometry>
 	    </collision>
 	    <visual>
-	      <origin xyz="0 0 0.1" rpy="0 0 0"/>
+	      <origin xyz="0 0 0.05" rpy="0 0 0"/>
 	      <geometry>
-		<box size="0.05 0.05 0.25"/>
+		<box size="0.05 0.05 0.15"/>
 	      </geometry>
 	      <material name="red">
@@ -161,5 +161,5 @@
   <joint name="camera_joint" type="continuous">
 	    <axis xyz="0 0 1" />
-	    <origin xyz="0 0 0.27" rpy="0 0 0"/>
+	    <origin xyz="0 0 0.15" rpy="0 0 0"/>
 	    <parent link="camera_link_connection"/>
 	    <child link="camera_link"/>
